File: Biifröst.kicad_pcb (KiCad board)
At the start: 2 copper layers, 42 x 84 mm, 15 parts, among them J1 Pitaya_Go, J2 LCD_SPI, J3 SPI_SD, J4 CMSIS-DAP, J5 DEBUG UART *DNP*, SW1 JS1400AFQ, SW2 TL9100AF200Q, SW3 TL9100AF200Q

Commit message: Add Wordmark/Icon for flair.
Parts:
- added Ref**: Val**, Biifröst:Horn_of_Odin, F.Cu at (21.0, 44.0)
- added Ref**: Val**, Biifröst:Logo, B.Cu at (21.6, 45.7)
- added Ref**: Val**, Biifröst:Wordmark, B.Cu at (28.0, 44.5)
